Commit message: fix 「no ros2_control tag」error

File: manipulator_description/urdf/manipulator.urdf.xacro (robot description, xacro)
@@ -31,3 +31,17 @@
     </visual>
   </link>
+  <xacro:property name="NAME_JOINT_0" value="joint0"/>
+  <xacro:property name="NAME_JOINT_1" value="joint1"/>
+  <xacro:property name="JOINT_0_LOWER_LIMIT" value="-70"/>
+  <xacro:property name="JOINT_0_UPPER_LIMIT" value="70"/>
+  <xacro:property name="JOINT_1_LOWER_LIMIT" value="-70"/>
+  <xacro:property name="JOINT_1_UPPER_LIMIT" value="70"/>
+  <xacro:manipulator_ros2_control_settings
+    name="manipulator"
+    name_joint_0="${name_joint_0}"
+    name_joint_1="${NAME_JOINT_1}"
+    joint_0_lower_limit="${JOINT_0_LOWER_LIMIT}"
+    joint_0_upper_limit="${JOINT_0_UPPER_LIMIT}"
+    joint_1_lower_limit="${JOINT_1_LOWER_LIMIT}"
+    joint_1_upper_limit="${JOINT_1_UPPER_LIMIT}" />
 </robot>

Commit message: add meshes data

File: manipulator_description/urdf/manipulator.urdf.xacro (robot description, xacro)
@@ -2,5 +2,34 @@
 <robot xmlns:xacro="http://www.ros.org/wiki/xacro" name="manipulator">
   <xacro:include filename="$(find manipulator_description)/urdf/manipulator.ros2_control.xacro"/>
-  <link name="base_link"></link>
+  <xacro:property name="MESH_BASE_LINK" value="manipulator_description/meshes/visual/base_link.stl"/>
+  <xacro:property name="MESH_LINK_1" value="manipulator_description/meshes/visual/link1.stl"/>
+  <xacro:property name="MESH_CAMERA_LINK" value="manipulator_description/meshes/visual/camera_link.stl"/>
+  <xacro:property name="MESH_COLLISION_BASE_LINK" value="manipulator_description/meshes/collision/base_link.stl"/>
+  <xacro:property name="MESH_LINK_1" value="manipulator_description/meshes/collision/link1.stl"/>
+  <xacro:property name="MESH_COLLISION_CAMERA_LINK" value="manipulator_description/meshes/collision/camera_link.stl"/>
+  <material name="black">
+    <color rgba="0.2 0.2 0.2 1.0"/>
+  </material>
+  <material name="red">
+    <color rgba=".8 0 0 1"/>
+  </material>
+  <link name="base_link">
+    <visual>
+        <origin xyz="0 0 0" rpy="0 0 0"/>
+        <geometry>
+          <mesh filename="package://${MESH_BASE_LINK}"
+              scale="1 1 1"/>
+        </geometry>
+        <material name="black"/>
+      </visual>
+      <collision>
+        <origin xyz="0 0 0" rpy="0 0 0"/>
+        <geometry>
+          <mesh filename="package://${MESH_COLLISION_BASE_LINK}"
+              scale="1 1 1"/>
+        </geometry>
+        <material name="black"/>
+      </collision>
+  </link>
   <joint name="joint0" type="continuous">
     <parent link="base_link"/>
@@ -10,5 +39,22 @@
     <limit effort="0.5" velocity="6.0" />
   </joint>
-  <link name="link1"></link>
+  <link name="link1">
+    <visual>
+      <origin xyz="0 0 0" rpy="0 0 0"/>
+      <geometry>
+        <mesh filename="package://${MESH_LINK_1}"
+            scale="1 1 1"/>
+      </geometry>
+      <material name="black"/>
+    </visual>
+    <collision>
+      <origin xyz="0 0 0" rpy="0 0 0"/>
+      <geometry>
+        <mesh filename="package://${MESH_COLLISION_LINK_1}"
+            scale="1 1 1"/>
+      </geometry>
+      <material name="black"/>
+    </collision>
+  </link>
   <joint name="joint1" type="continuous">
     <parent link="link1"/>
@@ -20,14 +66,21 @@
     <dynamics damping="0.4" />
   </joint>
-   <link name="camera_link">
+  <link name="camera_link">
     <visual>
-      <origin xyz="0 0 0.0125" rpy="0 0 0" />
+      <origin xyz="0 0 0.0125" rpy="0 0 0"/>
       <geometry>
-        <box size="0.05 0.045 0.025" />
+        <mesh filename="package://${MESH_CAMERA_LINK}"
+            scale="1 1 1"/>
       </geometry>
-      <material name="red">
-        <color rgba=".8 0 0 1" />
-      </material>
+      <material name="black"/>
     </visual>
+    <collision>
+      <origin xyz="0 0 0.0125" rpy="0 0 0"/>
+      <geometry>
+        <mesh filename="package://${MESH_COLLISION_CAMERA_LINK}"
+            scale="1 1 1"/>
+      </geometry>
+      <material name="black"/>
+    </collision>
   </link>
   <xacro:property name="NAME_JOINT_0" value="joint0"/>

Commit message: fix mesh file path

File: manipulator_description/urdf/manipulator.urdf.xacro (robot description, xacro)
@@ -6,5 +6,5 @@
   <xacro:property name="MESH_CAMERA_LINK" value="manipulator_description/meshes/visual/camera_link.stl"/>
   <xacro:property name="MESH_COLLISION_BASE_LINK" value="manipulator_description/meshes/collision/base_link.stl"/>
-  <xacro:property name="MESH_LINK_1" value="manipulator_description/meshes/collision/link1.stl"/>
+  <xacro:property name="MESH_COLLISION_LINK_1" value="manipulator_description/meshes/collision/link1.stl"/>
   <xacro:property name="MESH_COLLISION_CAMERA_LINK" value="manipulator_description/meshes/collision/camera_link.stl"/>
   <material name="black">
